File: hardware/flappy-esp32c3.kicad_pcb (KiCad board)
At the start: 2 copper layers, 90 x 60 mm, 55 parts, among them J1 USB-C-Breakout 16P, J2 LiPo 1S 500 mAh, J3 OLED SSD1306 SPI, J4 Arcade-Taster, SW1 Ein/Aus, U1 ESP32-C3-WROOM-02-N4, U2 MCP73831-2-OT, U3 AP2112K-3.3

Commit message: .
Routing:
- net LED_CHG: track 30.5 -> 21.0 mm
- net PROG: track 14.7 -> 9.24 mm
- net +3V3_MCU: track 126.0 -> 125.1 mm
