File: hardware/flappy-esp32c3.kicad_pcb (KiCad board)
At the start: 2 copper layers, 90 x 60 mm, 55 parts, among them J1 USB-C-Breakout 16P, J2 LiPo 1S 500 mAh, J3 OLED SSD1306 SPI, J4 Arcade-Taster, SW1 Ein/Aus, U1 ESP32-C3-WROOM-02-N4, U2 MCP73831-2-OT, U3 AP2112K-3.3

Commit message: update
Parts:
- removed LS1: Piezo 12 mm, Buzzer_Beeper:Buzzer_12x9.5RM7.6
- added J5: Piezo CEP-1114, Connector_JST:JST_XH_B2B-XH-A_1x02_P2.50mm_Vertical, F.Cu at (42.0, 60.0)
- added R17: 5k1, Resistor_SMD:R_0805_2012Metric_Pad1.20x1.40mm_HandSolder, F.Cu at (50.0, 44.0)
- added R18: 5k1, Resistor_SMD:R_0805_2012Metric_Pad1.20x1.40mm_HandSolder, F.Cu at (50.0, 46.5)
- C1: value 4u7 -> 4u7 25V X7R
- C10, C11, C2, C4, C7, C9: value 100n -> 100n 50V X7R
- C3: value 4u7 -> 10u 25V X7R
- C5: value 1u -> 2u2 16V X7R
- C6: value 22u -> 22u 10V X5R
- C8: value 10u -> 10u 16V X7R
- R14: value 1k -> 330R
- R2: value 1k -> 560R
- U2: value MCP73831-2-OT -> MCP73831T-2ACI/OT
Connections:
- J1 pad 5: unconnected-(J1-Pin_5-Pad5) -> USB_CC1
- J1 pad 6: unconnected-(J1-Pin_6-Pad6) -> USB_CC2
Routing:
- net BUZZ: track 25.6 -> 69.4 mm
- net +3V3_MCU: track 125.1 -> 108.1 mm, vias 6 -> 12
- net USB_CC1: track 0.00 -> 16.8 mm, vias 0 -> 2
- net USB_CC2: track 0.00 -> 7.96 mm, vias 0 -> 2
- net LED_G: track 53.1 -> 56.5 mm
- net BUZZ_P: track 14.7 -> 16.9 mm
- net USB_DM: track 34.1 -> 35.3 mm
- net OLED_CS: track 28.2 -> 29.1 mm, vias 2 -> 4
- net BTN: track 31.2 -> 30.3 mm
- net GND: track 11.3 -> 12.0 mm, vias 82 -> 88
Other:
- board text added: "J5 Piezo: 1 = +, 2 = - (CEP-1114 sitzt am Kabel)"
- board text added: "PIEZO"
- board text added: "R17/R18 nur bestuecken, wenn Breakout ohne 5k1-Rd"

Commit message: .
Parts:
- added C12: 100n 50V X7R, Capacitor_SMD:C_0805_2012Metric_Pad1.18x1.45mm_HandSolder, F.Cu at (76.0, 63.0)
- added D5: USBLC6-2SC6, Package_TO_SOT_SMD:SOT-23-6_Handsoldering, F.Cu at (52.0, 66.0)
- added R19: 1M, Resistor_SMD:R_0805_2012Metric_Pad1.20x1.40mm_HandSolder, F.Cu at (108.0, 57.0)
- added R20: 100k, Resistor_SMD:R_0805_2012Metric_Pad1.20x1.40mm_HandSolder, F.Cu at (50.0, 54.0)
- added R21: 100k, Resistor_SMD:R_0805_2012Metric_Pad1.20x1.40mm_HandSolder, F.Cu at (55.0, 54.0)
- added R22: 1M, Resistor_SMD:R_0805_2012Metric_Pad1.20x1.40mm_HandSolder, F.Cu at (66.0, 63.0)
- added R23: 1M, Resistor_SMD:R_0805_2012Metric_Pad1.20x1.40mm_HandSolder, F.Cu at (71.0, 63.0)
- J3: footprint Connector_JST:JST_XH_B7B-XH-A_1x07_P2.50mm_Vertical -> Connector_JST:JST_XH_B8B-XH-A_1x08_P2.50mm_Vertical
Connections:
- C5 pad 1: VBAT_SW -> VBAT
- J3 pad 4: MOSI -> GND
- J3 pad 5: OLED_RES -> MOSI
- J3 pad 6: OLED_DC -> OLED_RES
- J3 pad 7: OLED_CS -> OLED_DC
- SW1 pad 1: VBAT_SW -> LDO_EN
- U1 pad 10: unconnected-(U1-IO10-Pad10) -> LED_G
- U1 pad 11: unconnected-(U1-IO20/RXD-Pad11) -> VBUS_SENSE
- U1 pad 18: LED_G -> VBAT_SENSE
- U3 pad 1: VBAT_SW -> VBAT
- U3 pad 3: VBAT_SW -> LDO_EN
Routing:
- net VBAT_SENSE: track 0.00 -> 104.5 mm, vias 0 -> 4
- net VBAT: track 43.7 -> 106.8 mm
- net LDO_EN: track 0.00 -> 57.0 mm, vias 0 -> 4
- net VBAT_SW: track 41.8 -> 0.00 mm
- net LED_G: track 56.5 -> 19.0 mm, vias 0 -> 6
- net USB_DM: track 35.3 -> 71.5 mm, vias 2 -> 4
- net BTN_CON: track 10.9 -> 42.7 mm, vias 0 -> 2
- net VBUS_SENSE: track 0.00 -> 31.6 mm, vias 0 -> 8
- net BUZZ_P: track 16.9 -> 29.9 mm, vias 2 -> 4
- net USB_CC1: track 16.8 -> 7.14 mm
- net VBUS: track 59.0 -> 68.6 mm
- net OLED_RES: track 27.3 -> 34.4 mm, vias 2 -> 4
- net EN: track 27.0 -> 32.0 mm, vias 2 -> 8
- net MOSI: track 23.0 -> 27.2 mm, vias 2 -> 4
- net OLED_DC: track 25.4 -> 28.5 mm, vias 2 -> 4
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Other:
- board text added: "D5: ESD-Klemme Taster + Piezo"
- board text added: "J3 Display: 1 GND 2 VCC 3 SCLK 4 GND 5 MOSI 6 RES 7 DC 8 CS"
- board text removed: "J3 Display: 1 GND 2 VCC 3 SCLK 4 MOSI 5 RES 6 DC 7 CS"
